File: hardware/kicad/BBB_SensorCape.kicad_pcb (KiCad board)
At the start: 2 copper layers, 86.4 x 54.6 mm, 58 parts, among them P8 CONN_23X2, P9 CONN_23X2, SW1 SW_IT11095S, SW2 SW_IT11095S, SW3 SW_IT11095S, SW4 SW_IT11095S, SW5 DIPS_02, U1 MPU-9150, U2 TMP006, U3 BMP-180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

Commit message: Added files for hardware version 0.9
Parts:
- removed C13, C18, C19: 100n, SM0805
- removed C20: 220n, SM0805
- removed D2, D3, D4: ORANGE, LED-0805
- removed JP1, JP2, JP3, JP4: JUMPER, PIN_ARRAY_2X1
- removed PAD_15milx15mil: VAL**, PAD_15milx15mil
- removed R11, R12, R13, R14: 820, SM0805
- removed R17, R18: 10k, SM0805
- removed SW3, SW4: SW_IT11095S, SW_IT11095S
- added LOGO: , LOGO, F.Cu at (68.1, 57.9)
- added P1: CONN_2, BAT_CR1216, B.Cu at (77.3, 42.2)
- added Q1: MMBT3904, sot23, F.Cu at (29.6, 20.1)
- added R2: 120, SM0805, F.Cu at (32.4, 21.1)
- added R3: 10k, SM0805, F.Cu at (76.8, 23.6)
- D1: value ORANGE -> TSAL4400; footprint LED-0805 -> LED-3MM
- R7, R8, R9: value 4.75k -> 4.7k
- SW1, SW2: footprint SW_IT11095S -> FSM4JH
- U5: value CHIPCAP2 -> MCP79410; footprint CHIPCAP2 -> so-8
- moved C15 50.0 mm to (63.2, 22.5), turned to 0 degrees
- moved R7 45.8 mm to (63.2, 26.2), turned to 180 degrees
- moved SW1 45.7 mm to (41.4, 43.9), turned to 180 degrees
- moved SW2 45.3 mm to (41.4, 37.1), turned to 180 degrees
- moved R10 44.7 mm to (63.2, 24.3), turned to 0 degrees
- moved R9 44.5 mm to (63.2, 30.0), turned to 180 degrees
- moved R8 43.1 mm to (63.2, 28.1), turned to 180 degrees
- moved C16 42.1 mm to (47.4, 43.1), turned to 0 degrees
- moved R16 40.9 mm to (47.4, 38.0)
- moved SW5 40.5 mm to (56.1, 32.6)
- moved C17 39.5 mm to (47.4, 36.1)
- moved U7 39.3 mm to (57.5, 24.5)
- moved R15 39.2 mm to (47.4, 45.0), turned to 180 degrees
- moved C14 37.1 mm to (29.6, 29.5), turned to 180 degrees
- moved R6 36.7 mm to (29.6, 27.6)
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Connections:
- C1 pad 1: 3V3B -> +3.3V
- C1 pad 2: AGND -> DGND
- C10 pad 1: 3V3B -> +3.3V
- C10 pad 2: AGND -> DGND
- C11 pad 1: 3V3B -> 3V3
- C11 pad 2: AGND -> DGND
- C12 pad 1: 3V3B -> 3V3
- C12 pad 2: AGND -> DGND
- C14 pad 1: AGND -> DGND
- C15 pad 1: 3V3B -> 3V3
- C15 pad 2: AGND -> DGND
- C16 pad 1: JP1 -> SW1
- C16 pad 2: AGND -> DGND
- C17 pad 1: JP2 -> SW2
- C17 pad 2: AGND -> DGND
- C2 pad 2: AGND -> DGND
- C3 pad 1: 3V3B -> 3V3
- C3 pad 2: AGND -> DGND
- C4 pad 1: AGND -> N-0000030
- C4 pad 2: N-0000029 -> DGND
- C5 pad 1: 3V3B -> 3V3
- C5 pad 2: AGND -> DGND
- C9 pad 1: AGND -> 3V3
- C9 pad 2: 3V3B -> DGND
- D1 pad 1: N-000004 -> +5V
- D1 pad 2: AGND -> N-0000023
- P8 pad 1: AGND -> DGND
- P8 pad 10: LED1 -> (no net)
- P8 pad 11: INT_LT -> (no net)
- P8 pad 17: AL -> (no net)
- P8 pad 19: AH -> (no net)
- P8 pad 2: AGND -> DGND
- P8 pad 7: LED3 -> (no net)
- P8 pad 8: LED4 -> (no net)
- P8 pad 9: LED2 -> IR
- P9 pad 1: AGND -> DGND
- P9 pad 11: IR -> (no net)
- P9 pad 14: (no net) -> IR_PWM
- P9 pad 2: AGND -> DGND
- P9 pad 22: INT_M -> (no net)
- P9 pad 23: SW2 -> SW1
- P9 pad 24: SW3 -> SW2
- P9 pad 25: SW1 -> INT_M
- P9 pad 26: SW4 -> INT_LT
- P9 pad 3: (no net) -> +3.3V
- P9 pad 4: 3V3B -> 3V3
- P9 pad 43: AGND -> DGND
- P9 pad 44: AGND -> DGND
- P9 pad 45: AGND -> DGND
- P9 pad 46: AGND -> DGND
- P9 pad 6: (no net) -> +5V
- R1 pad 2: 3V3B -> 3V3
- R10 pad 2: 3V3B -> 3V3
- R15 pad 1: 3V3B -> +3.3V
- R15 pad 2: JP1 -> SW1
- R16 pad 1: 3V3B -> +3.3V
- R16 pad 2: JP2 -> SW2
- R21 pad 2: 3V3B -> +3.3V
- R22 pad 2: 3V3B -> +3.3V
- R4 pad 2: AGND -> DGND
- R5 pad 1: 3V3B -> +3.3V
- R6 pad 2: 3V3B -> 3V3
- R7 pad 1: 3V3B -> N-0000039
- R7 pad 2: N-0000011 -> 3V3
- R8 pad 1: 3V3B -> N-0000038
- R8 pad 2: N-0000012 -> 3V3
- R9 pad 1: 3V3B -> N-0000011
- R9 pad 2: N-0000013 -> 3V3
- SW1 pad 1: AGND -> DGND
- SW1 pad 2: AGND -> DGND
- SW1 pad 3: JP1 -> SW1
- SW1 pad 4: JP1 -> SW1
- SW2 pad 1: AGND -> DGND
- SW2 pad 2: AGND -> DGND
- SW2 pad 3: JP2 -> SW2
- SW2 pad 4: JP2 -> SW2
- SW5 pad 1: N-0000013 -> N-0000039
- SW5 pad 2: N-0000012 -> N-0000038
- SW5 pad 3: AGND -> DGND
- SW5 pad 4: AGND -> DGND
- U1 pad 1: AGND -> (no net)
- U1 pad 11: AGND -> DGND
- U1 pad 13: 3V3B -> 3V3
- U1 pad 15: AGND -> DGND
- U1 pad 17: AGND -> DGND
- U1 pad 18: AGND -> DGND
- U1 pad 20: N-0000029 -> N-0000030
- U1 pad 3: 3V3B -> 3V3
- U1 pad 8: 3V3B -> +3.3V
- U1 pad 9: AGND -> DGND
- U2 pad A1: AGND -> DGND
- U2 pad A2: AGND -> DGND
- U2 pad A3: 3V3B -> 3V3
- U2 pad B1: AGND -> DGND
- U2 pad C1: 3V3B -> 3V3
- U3 pad 2: 3V3B -> 3V3
- U3 pad 3: 3V3B -> +3.3V
- U3 pad 7: AGND -> DGND
- U4 pad 1: 3V3B -> 3V3
- U4 pad 2: AGND -> DGND
- U5 pad 1: AL -> N-0000017
- U5 pad 2: (no net) -> N-0000018
- U5 pad 3: I2C_SDA_2 -> N-0000022
- U5 pad 4: I2C_SCL_2 -> DGND
- U5 pad 5: N-0000019 -> I2C_SDA_2
- U5 pad 6: AGND -> I2C_SCL_2
- U5 pad 7: 3V3B -> N-0000024
- U5 pad 8: AH -> 3V3
- U6 pad 2: AGND -> DGND
- U7 pad 1: N-0000013 -> N-0000039
- U7 pad 2: N-0000012 -> N-0000038
- U7 pad 4: AGND -> DGND
- U7 pad 8: 3V3B -> 3V3
Routing:
- net AGND: track 374.3 -> 0.00 mm, vias 23 -> 0
- net 3V3B: track 365.1 -> 0.00 mm, vias 19 -> 0
- net 3V3: track 0.00 -> 176.1 mm, vias 0 -> 10
- net +3.3V: track 0.00 -> 134.9 mm, vias 0 -> 10
- net I2C_SDA_2: track 93.5 -> 162.6 mm, vias 10 -> 12
- net +5V: track 0.00 -> 59.7 mm
- net IR_PWM: track 0.00 -> 59.6 mm, vias 0 -> 1
- net JP3: track 40.9 -> 0.00 mm
- net SW3: track 39.4 -> 0.00 mm
- net I2C_SCL_2: track 100.4 -> 133.9 mm
- net LED1: track 28.7 -> 0.00 mm
- net N-0000039: track 0.00 -> 28.4 mm, vias 0 -> 2
- net SW1: track 20.8 -> 43.7 mm, vias 0 -> 1
- net DGND: track 0.00 -> 22.2 mm, vias 0 -> 6
- net LED2: track 21.7 -> 0.00 mm
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- added copper zone on F.Cu, net DGND
- added copper zone on B.Cu, net N-0000022
- removed copper zone on B.Cu, net AGND
- removed copper zone on F.Cu, net AGND
Other:
- outline, holes or cut-outs redrawn
- board text added: "DC: 072513"
- board text added: "IR Rx."
- board text added: "IR Tx."
- board text added: "Rev. 0.9"
- board text removed: "1"
- board text removed: "2"
- board text removed: "3"
- board text removed: "4"
- board text removed: "BeagleBoard.org"
- board text removed: "DC: 063013"
- board text removed: "Humidity"
- board text removed: "IR"
- board text removed: "Rev. 0.2"
- board text removed: "User LEDs"
