File: hardware/kicad/BBB_SensorCape.sch (KiCad schematic (older format))
At the start: 53 parts, among them SW1 SW_IT11095S, SW2 SW_IT11095S, SW3 SW_IT11095S, SW4 SW_IT11095S, SW5 DIPS_02, U1 MPU-9150, U2 TMP006, U3 BMP-180, U4 ISL29023, U5 CHIPCAP2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

Commit message: Added files for hardware version 0.9
Parts:
- removed C13, C18, C19: 100n, ~, symbol C
- removed C20: 220n, ~, symbol C
- removed D2, D3, D4: ORANGE, ~, symbol LED
- removed JP1, JP2, JP3, JP4: JUMPER, ~, symbol JUMPER
- removed R11, R12, R13, R14: 820, ~, symbol R
- removed R17, R18: 10k, ~, symbol R
- removed SW3, SW4: SW_IT11095S, symbol SW_IT11095S
- removed U5: CHIPCAP2, ~, symbol CHIPCAP2
- added P1: CONN_2, symbol CONN_2
- added Q1: MMBT3904, ~, symbol NPN
- added R2: 120, ~, symbol R
- added R3: 10k, ~, symbol R
- added U5: MCP79410, symbol MCP79410
- added X1: CRYSTAL, ~, symbol CRYSTAL
- D1: value ORANGE -> TSAL4400
- R7, R8, R9: value 4.75k -> 4.7k
- SW1, SW2: footprint (none) -> FSM4JH
Connections:
- net labels added: +3,3V, +5V, 3V3, DGND, IR_PWM
- net labels removed: 3V3B, AGND, AH, AL, APWR, JP1, JP2, JP3, JP4, LED1, LED2, LED3, LED4, SW3, SW4
- wire segments 148 -> 145
- no-connect marks 3 -> 11
Other:
- note added: "IR Emitter"
- note added: "IR Reciever"
- note added: "Real Time Clock"
- note removed: "Humidity/Temperature Sensor"
- note removed: "IR Sensor"
- note removed: "User LED's"
- moved on the sheet: C1, C10, C11, C12, C14, C15, C16, C17, C2, C3, C5, C9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
